File: prok_smd/multi_power.kicad_pcb (KiCad board)
At the start: 2 copper layers, 38 x 79 mm, 17 parts, among them J1 Conn_01x03_Female, J2 Conn_01x05_Female, J3 Conn_01x03_Female, J4 Conn_01x05_Female, J5 Conn_01x05_Female, J6 Conn_01x03_Female, J7 POWER, J8 Conn_01x05_Female, J9 Conn_01x03_Female, U1 REG1117

Commit message: :recycle: redid power pcb single
Other:
- board size 38 x 79 mm -> 38 x 77 mm
Changed lines of the file:
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@@
-(kicad_pcb (version 20171130) (host pcbnew "(5.0.2)-1")
+(kicad_pcb (version 20171130) (host pcbnew "(5.1.5)-3")
   (general
     (thickness 1.6)
@@
     (zone_45_only no)
     (trace_min 0.127)
-    (segment_width 0.2)
-    (edge_width 0.2)
     (via_size 0.6)
     (via_drill 0.3)
@@
     (uvia_min_size 0.2)
     (uvia_min_drill 0.1)
+    (edge_width 0.2)
+    (segment_width 0.2)
     (pcb_text_width 0.3)
     (pcb_text_size 1.5 1.5)
@@
     (uvia_dia 0.3)
     (uvia_drill 0.1)
+    (diff_pair_width 0.127)
     (diff_pair_gap 0.127)
-    (diff_pair_width 0.127)
     (add_net +12V)
     (add_net +5V)
@@
   (gr_arc (start 98 123) (end 95 123) (angle -90) (layer Edge.Cuts) (width 0.2))
   (gr_arc (start 75 123) (end 75 126) (angle -90) (layer Edge.Cuts) (width 0.2))
-  (gr_line (start 107 50) (end 107 123) (layer Edge.Cuts) (width 0.15))
-  (gr_line (start 72 47) (end 104 47) (layer Edge.Cuts) (width 0.15))
-  (gr_line (start 69 50) (end 69 123) (layer Edge.Cuts) (width 0.15))
-  (gr_arc (start 72 50) (end 72 47) (angle -90) (layer Edge.Cuts) (width 0.15))
-  (gr_arc (start 104 50) (end 107 50) (angle -90) (layer Edge.Cuts) (width 0.15))
+  (gr_line (start 107 52) (end 107 123) (layer Edge.Cuts) (width 0.15))
+  (gr_line (start 72 49) (end 104 49) (layer Edge.Cuts) (width 0.15))
+  (gr_line (start 69 52) (end 69 123) (layer Edge.Cuts) (width 0.15))
+  (gr_arc (start 72 52) (end 72 49) (angle -90) (layer Edge.Cuts) (width 0.15))
+  (gr_arc (start 104 52) (end 107 52) (angle -90) (layer Edge.Cuts) (width 0.15))
   (gr_arc (start 104 123) (end 104 126) (angle -90) (layer Edge.Cuts) (width 0.15))
   (gr_arc (start 72 123) (end 69 123) (angle -90) (layer Edge.Cuts) (width 0.15))
