File: prok_smd/prok_smd.sch (KiCad schematic (older format))
At the start: 26 parts, among them J1 POWER, J10 Conn_01x04_Female, J11 Conn_01x04_Female, J2 EXPAND, J3 Conn_01x11, J4 Conn_01x07, J9 Conn_01x05_Female, U1 Teensy3.2, U2 MCP6002, U3 TL072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

Commit message: :construction: Locked headers and added mousebites
Parts:
- removed J10, J11: Conn_01x04_Female, Connector_PinSocket_2.54mm:PinSocket_1x04_P2.54mm_Vertical, symbol Connector:Conn_01x04_Female
- added HS1: Heatsink_Pad, symbol Mechanical:Heatsink_Pad
- added J10, J11, J13, J14: Conn_01x02_Female, Connector_PinSocket_2.54mm:PinSocket_1x02_P2.54mm_Vertical, symbol Connector:Conn_01x02_Female
Connections:
- net labels added: REG_HEAT
- wire segments 137 -> 138
- no-connect marks 28 -> 29
Changed lines of the file:
@@
 P 3850 5750
 F 0 "U4" H 3875 5965 50  0000 C CNN
-F 1 "REG1117" H 3875 5874 50  0000 C CNN
+F 1 "REG1117" H 3800 5850 50  0000 C CNN
 F 2 "Package_TO_SOT_SMD:SOT-223" H 3850 5750 50  0001 C CNN
 F 3 "" H 3850 5750 50  0001 C CNN
@@
 Connection ~ 5550 6300
 $Comp
-L Connector:Conn_01x04_Female J11
-U 1 1 5D1980FD
-P 5000 7350
-F 0 "J11" H 5027 7326 50  0000 L CNN
-F 1 "Conn_01x04_Female" H 5027 7235 50  0000 L CNN
-F 2 "Connector_PinSocket_2.54mm:PinSocket_1x04_P2.54mm_Vertical" H 5000 7350 50  0001 C CNN
-F 3 "~" H 5000 7350 50  0001 C CNN
-	1    5000 7350
-	1    0    0    -1
-$EndComp
-$Comp
-L Connector:Conn_01x04_Female J10
-U 1 1 5D19814F
-P 4400 7450
-F 0 "J10" H 4294 7025 50  0000 C CNN
-F 1 "Conn_01x04_Female" H 4294 7116 50  0000 C CNN
-F 2 "Connector_PinSocket_2.54mm:PinSocket_1x04_P2.54mm_Vertical" H 4400 7450 50  0001 C CNN
-F 3 "~" H 4400 7450 50  0001 C CNN
-	1    4400 7450
-	-1   0    0    1
-$EndComp
-$Comp
 L power:GND #PWR0135
 U 1 1 5D19822F
@@
 Connection ~ 4700 7550
 Wire Wire Line
-	4700 7550 4800 7550
-Wire Wire Line
-	4800 7450 4600 7450
-Wire Wire Line
-	4600 7350 4800 7350
-Wire Wire Line
-	4800 7250 4700 7250
+	4700 7550 4750 7550
+Wire Wire Line
+	4600 7350 4750 7350
 Wire Wire Line
 	4700 7250 4700 7550
@@
 L power:-12V #PWR0136
 U 1 1 5D1B34A3
-P 3000 7350
-F 0 "#PWR0136" H 3000 7450 50  0001 C CNN
-F 1 "-12V" H 3015 7523 50  0000 C CNN
-F 2 "" H 3000 7350 50  0001 C CNN
-F 3 "" H 3000 7350 50  0001 C CNN
-	1    3000 7350
+P 3000 7550
+F 0 "#PWR0136" H 3000 7650 50  0001 C CNN
+F 1 "-12V" H 3015 7723 50  0000 C CNN
+F 2 "" H 3000 7550 50  0001 C CNN
+F 3 "" H 3000 7550 50  0001 C CNN
+	1    3000 7550
 	0    -1   -1   0
 $EndComp
@@
 L power:+5V #PWR0139
 U 1 1 5D1B3758
-P 3000 7550
-F 0 "#PWR0139" H 3000 7400 50  0001 C CNN
-F 1 "+5V" V 3015 7678 50  0000 L CNN
-F 2 "" H 3000 7550 50  0001 C CNN
-F 3 "" H 3000 7550 50  0001 C CNN
-	1    3000 7550
+P 3000 7350
+F 0 "#PWR0139" H 3000 7200 50  0001 C CNN
+F 1 "+5V" V 3015 7478 50  0000 L CNN
+F 2 "" H 3000 7350 50  0001 C CNN
+F 3 "" H 3000 7350 50  0001 C CNN
+	1    3000 7350
 	0    -1   -1   0
 $EndComp
@@
 Wire Wire Line
 	3000 7550 3100 7550
+Text GLabel 10000 6000 0    50   Input ~ 0
+REG_HEAT
+NoConn ~ 10000 6000
+$Comp
+L Mechanical:Heatsink_Pad HS1
+U 1 1 5D1FCE37
+P 4200 5600
+F 0 "HS1" V 4153 5729 50  0000 L CNN
+F 1 "Heatsink_Pad" V 4244 5729 50  0000 L CNN
+F 2 "" H 4212 5550 50  0001 C CNN
+F 3 "~" H 4212 5550 50  0001 C CNN
+	1    4200 5600
+	0    1    1    0
+$EndComp
+Wire Wire Line
+	4100 5600 4050 5600
+$Comp
+L Connector:Conn_01x02_Female J13
+U 1 1 5D2044FC
+P 4950 7250
+F 0 "J13" H 4977 7226 50  0000 L CNN
+F 1 "Conn_01x02_Female" H 4977 7135 50  0000 L CNN
+F 2 "Connector_PinSocket_2.54mm:PinSocket_1x02_P2.54mm_Vertical" H 4950 7250 50  0001 C CNN
+F 3 "~" H 4950 7250 50  0001 C CNN
+	1    4950 7250
+	1    0    0    -1
+$EndComp
+$Comp
+L Connector:Conn_01x02_Female J14
+U 1 1 5D20455E
+P 4950 7450
+F 0 "J14" H 4977 7426 50  0000 L CNN
+F 1 "Conn_01x02_Female" H 4977 7335 50  0000 L CNN
+F 2 "Connector_PinSocket_2.54mm:PinSocket_1x02_P2.54mm_Vertical" H 4950 7450 50  0001 C CNN
+F 3 "~" H 4950 7450 50  0001 C CNN
+	1    4950 7450
+	1    0    0    -1
+$EndComp
+$Comp
+L Connector:Conn_01x02_Female J10
+U 1 1 5D2045BC
+P 4400 7350
+F 0 "J10" H 4294 7025 50  0000 C CNN
+F 1 "Conn_01x02_Female" H 4294 7116 50  0000 C CNN
+F 2 "Connector_PinSocket_2.54mm:PinSocket_1x02_P2.54mm_Vertical" H 4400 7350 50  0001 C CNN
+F 3 "~" H 4400 7350 50  0001 C CNN
+	1    4400 7350
+	-1   0    0    1
+$EndComp
+$Comp
+L Connector:Conn_01x02_Female J11
+U 1 1 5D204674
+P 4400 7550
+F 0 "J11" H 4294 7225 50  0000 C CNN
+F 1 "Conn_01x02_Female" H 4294 7316 50  0000 C CNN
+F 2 "Connector_PinSocket_2.54mm:PinSocket_1x02_P2.54mm_Vertical" H 4400 7550 50  0001 C CNN
+F 3 "~" H 4400 7550 50  0001 C CNN
+	1    4400 7550
+	-1   0    0    1
+$EndComp
+Wire Wire Line
+	4750 7250 4700 7250
+Wire Wire Line
+	4750 7450 4600 7450
 $EndSCHEMATC

Commit message: :construction: first draft routing
Connections:
- wire segments 138 -> 142
Changed lines of the file:
@@
 	4700 7550 4750 7550
 Wire Wire Line
-	4600 7350 4750 7350
-Wire Wire Line
-	4700 7250 4700 7550
+	4700 7250 4700 7350
 Connection ~ 4700 7250
 Wire Wire Line
@@
 	4750 7250 4700 7250
 Wire Wire Line
-	4750 7450 4600 7450
+	4600 7350 4700 7350
+Connection ~ 4700 7350
+Wire Wire Line
+	4700 7350 4700 7450
+Wire Wire Line
+	4700 7350 4750 7350
+Wire Wire Line
+	4600 7450 4700 7450
+Connection ~ 4700 7450
+Wire Wire Line
+	4700 7450 4700 7550
+Wire Wire Line
+	4700 7450 4750 7450
 $EndSCHEMATC

Commit message: :sparkles: :construction: first draft v2 board
Parts:
- removed J10, J11, J13, J14: Conn_01x02_Female, Connector_PinSocket_2.54mm:PinSocket_1x02_P2.54mm_Vertical, symbol Connector:Conn_01x02_Female
- removed J3: Conn_01x11, symbol Connector_Generic:Conn_01x11
- removed J4: Conn_01x07, symbol Connector_Generic:Conn_01x07
- added J2: Conn_01x03_Female, Connector_PinSocket_2.54mm:PinSocket_1x03_P2.54mm_Vertical_SMD_Pin1Left, symbol Connector:Conn_01x03_Female
- J9: footprint Connector_PinSocket_2.54mm:PinSocket_1x05_P2.54mm_Vertical -> Connector_PinSocket_2.54mm:PinSocket_1x05_P2.54mm_Vertical_SMD_Pin1Left
- renumbered J2 to EXPAND1
Connections:
- net labels removed: REG_HEAT
- wire segments 142 -> 119
- no-connect marks 29 -> 28
Changed lines of the file:
@@
 NoConn ~ 4500 1700
 $Comp
-L Connector_Generic:Conn_02x03_Odd_Even J2
+L Connector_Generic:Conn_02x03_Odd_Even EXPAND1
 U 1 1 5D182574
 P 8150 1000
-F 0 "J2" H 8200 1317 50  0000 C CNN
+F 0 "EXPAND1" H 8200 1317 50  0000 C CNN
 F 1 "EXPAND" H 8200 1226 50  0000 C CNN
 F 2 "Connector_PinHeader_2.54mm:PinHeader_2x03_P2.54mm_Vertical" H 8150 1000 50  0001 C CNN
@@
 	3550 5850 3400 5850
 Connection ~ 3400 5850
-Text GLabel 9300 1700 0    50   Input ~ 0
-MISO
-Text GLabel 9300 1800 0    50   Input ~ 0
-LED_RESET
-Text GLabel 9300 1900 0    50   Input ~ 0
-SS
-Text GLabel 9300 2000 0    50   Input ~ 0
-RESET_CV
-Text GLabel 9300 2100 0    50   Input ~ 0
-RESET_SW
-Text GLabel 9300 2200 0    50   Input ~ 0
-MOSI
-Text GLabel 9300 2300 0    50   Input ~ 0
-LED_4
-Text GLabel 9300 2400 0    50   Input ~ 0
-LED_3
-Text GLabel 9300 2500 0    50   Input ~ 0
-LED_2
-Text GLabel 9300 2600 0    50   Input ~ 0
-LED_1
-$Comp
-L power:GND #PWR0119
-U 1 1 5D20EBAB
-P 9300 2700
-F 0 "#PWR0119" H 9300 2450 50  0001 C CNN
-F 1 "GND" V 9305 2572 50  0000 R CNN
-F 2 "" H 9300 2700 50  0001 C CNN
-F 3 "" H 9300 2700 50  0001 C CNN
-	1    9300 2700
-	0    1    1    0
-$EndComp
-Text GLabel 9300 3050 0    50   Input ~ 0
-TIME_CV
-Text GLabel 9300 3150 0    50   Input ~ 0
-CHANNEL_CV
-Text GLabel 9300 3250 0    50   Input ~ 0
-AUDIO_OUT
-$Comp
-L power:+3.3V #PWR0120
-U 1 1 5D20ED65
-P 9300 3350
-F 0 "#PWR0120" H 9300 3200 50  0001 C CNN
-F 1 "+3.3V" V 9315 3478 50  0000 L CNN
-F 2 "" H 9300 3350 50  0001 C CNN
-F 3 "" H 9300 3350 50  0001 C CNN
-	1    9300 3350
-	0    -1   -1   0
-$EndComp
-Text GLabel 9300 3450 0    50   Input ~ 0
-SCLK
-Text GLabel 9300 3550 0    50   Input ~ 0
-TIME_POT
-Text GLabel 9300 3650 0    50   Input ~ 0
-CHANNEL_POT
-$Comp
-L Connector_Generic:Conn_01x11 J3
-U 1 1 5D20F0C8
-P 9650 2200
-F 0 "J3" H 9569 1475 50  0000 C CNN
-F 1 "Conn_01x11" H 9569 1566 50  0000 C CNN
-F 2 "" H 9650 2200 50  0001 C CNN
-F 3 "~" H 9650 2200 50  0001 C CNN
-	1    9650 2200
-	1    0    0    1
-$EndComp
-Wire Wire Line
-	9450 1700 9300 1700
-Wire Wire Line
-	9300 1800 9450 1800
-Wire Wire Line
-	9450 1900 9300 1900
-Wire Wire Line
-	9300 2000 9450 2000
-Wire Wire Line
-	9450 2100 9300 2100
-Wire Wire Line
-	9300 2200 9450 2200
-Wire Wire Line
-	9450 2300 9300 2300
-Wire Wire Line
-	9300 2400 9450 2400
-Wire Wire Line
-	9450 2500 9300 2500
-Wire Wire Line
-	9300 2600 9450 2600
-Wire Wire Line
-	9450 2700 9300 2700
-$Comp
-L Connector_Generic:Conn_01x07 J4
-U 1 1 5D23CAC6
-P 9650 3350
-F 0 "J4" H 9569 2825 50  0000 C CNN
-F 1 "Conn_01x07" H 9569 2916 50  0000 C CNN
-F 2 "" H 9650 3350 50  0001 C CNN
-F 3 "~" H 9650 3350 50  0001 C CNN
-	1    9650 3350
-	1    0    0    1
-$EndComp
-Wire Wire Line
-	9300 3050 9450 3050
-Wire Wire Line
-	9450 3150 9300 3150
-Wire Wire Line
-	9300 3250 9450 3250
-Wire Wire Line
-	9450 3350 9300 3350
-Wire Wire Line
-	9300 3450 9450 3450
-Wire Wire Line
-	9450 3550 9300 3550
-Wire Wire Line
-	9300 3650 9450 3650
 $Sheet
 S 1400 1300 1250 1300
@@
 $EndComp
 Wire Wire Line
-	4600 7550 4700 7550
-Connection ~ 4700 7550
-Wire Wire Line
-	4700 7550 4750 7550
-Wire Wire Line
 	4700 7250 4700 7350
 Connection ~ 4700 7250
@@
 F 0 "J9" H 3327 7376 50  0000 L CNN
 F 1 "Conn_01x05_Female" H 3327 7285 50  0000 L CNN
-F 2 "Connector_PinSocket_2.54mm:PinSocket_1x05_P2.54mm_Vertical" H 3300 7350 50  0001 C CNN
+F 2 "Connector_PinSocket_2.54mm:PinSocket_1x05_P2.54mm_Vertical_SMD_Pin1Left" H 3300 7350 50  0001 C CNN
 F 3 "~" H 3300 7350 50  0001 C CNN
 	1    3300 7350
@@
 Wire Wire Line
 	3000 7550 3100 7550
-Text GLabel 10000 6000 0    50   Input ~ 0
-REG_HEAT
-NoConn ~ 10000 6000
 $Comp
 L Mechanical:Heatsink_Pad HS1
@@
 Wire Wire Line
 	4100 5600 4050 5600
-$Comp
-L Connector:Conn_01x02_Female J13
-U 1 1 5D2044FC
-P 4950 7250
-F 0 "J13" H 4977 7226 50  0000 L CNN
-F 1 "Conn_01x02_Female" H 4977 7135 50  0000 L CNN
-F 2 "Connector_PinSocket_2.54mm:PinSocket_1x02_P2.54mm_Vertical" H 4950 7250 50  0001 C CNN
-F 3 "~" H 4950 7250 50  0001 C CNN
-	1    4950 7250
-	1    0    0    -1
-$EndComp
-$Comp
-L Connector:Conn_01x02_Female J14
-U 1 1 5D20455E
-P 4950 7450
-F 0 "J14" H 4977 7426 50  0000 L CNN
-F 1 "Conn_01x02_Female" H 4977 7335 50  0000 L CNN
-F 2 "Connector_PinSocket_2.54mm:PinSocket_1x02_P2.54mm_Vertical" H 4950 7450 50  0001 C CNN
-F 3 "~" H 4950 7450 50  0001 C CNN
-	1    4950 7450
-	1    0    0    -1
-$EndComp
-$Comp
-L Connector:Conn_01x02_Female J10
-U 1 1 5D2045BC
-P 4400 7350
-F 0 "J10" H 4294 7025 50  0000 C CNN
-F 1 "Conn_01x02_Female" H 4294 7116 50  0000 C CNN
-F 2 "Connector_PinSocket_2.54mm:PinSocket_1x02_P2.54mm_Vertical" H 4400 7350 50  0001 C CNN
-F 3 "~" H 4400 7350 50  0001 C CNN
-	1    4400 7350
-	-1   0    0    1
-$EndComp
-$Comp
-L Connector:Conn_01x02_Female J11
-U 1 1 5D204674
-P 4400 7550
-F 0 "J11" H 4294 7225 50  0000 C CNN
-F 1 "Conn_01x02_Female" H 4294 7316 50  0000 C CNN
-F 2 "Connector_PinSocket_2.54mm:PinSocket_1x02_P2.54mm_Vertical" H 4400 7550 50  0001 C CNN
-F 3 "~" H 4400 7550 50  0001 C CNN
-	1    4400 7550
-	-1   0    0    1
-$EndComp
-Wire Wire Line
-	4750 7250 4700 7250
 Wire Wire Line
 	4600 7350 4700 7350
 Connection ~ 4700 7350
-Wire Wire Line
-	4700 7350 4700 7450
-Wire Wire Line
-	4700 7350 4750 7350
-Wire Wire Line
-	4600 7450 4700 7450
-Connection ~ 4700 7450
-Wire Wire Line
-	4700 7450 4700 7550
-Wire Wire Line
-	4700 7450 4750 7450
+$Comp
+L Connector:Conn_01x03_Female J2
+U 1 1 5D1D79FB
+P 4400 7250
+F 0 "J2" H 4294 6925 50  0000 C CNN
+F 1 "Conn_01x03_Female" H 4294 7016 50  0000 C CNN
+F 2 "Connector_PinSocket_2.54mm:PinSocket_1x03_P2.54mm_Vertical_SMD_Pin1Left" H 4400 7250 50  0001 C CNN
+F 3 "~" H 4400 7250 50  0001 C CNN
+	1    4400 7250
+	-1   0    0    1
+$EndComp
+Wire Wire Line
+	4700 7250 4700 7150
+Wire Wire Line
+	4600 7150 4700 7150
+Wire Wire Line
+	4700 7350 4700 7550
 $EndSCHEMATC

Commit message: :recycle: redid power pcb single
Parts:
- J2: value Conn_01x03_Female -> Conn_01x05_Female; footprint Connector_PinSocket_2.54mm:PinSocket_1x03_P2.54mm_Vertical_SMD_Pin1Left -> Connector_PinSocket_2.54mm:PinSocket_1x05_P2.54mm_Vertical_SMD_Pin1Left; symbol Connector:Conn_01x03_Female -> Connector:Conn_01x05_Female
Connections:
- net GND: now also J2.4 (Pin_4), J2.5 (Pin_5)
Changed lines of the file:
@@
 EESchema Schematic File Version 4
-LIBS:prok_smd-cache
-EELAYER 26 0
+EELAYER 30 0
 EELAYER END
 $Descr A4 11693 8268
@@
 	4600 7350 4700 7350
 Connection ~ 4700 7350
-$Comp
-L Connector:Conn_01x03_Female J2
+Wire Wire Line
+	4700 7250 4700 7150
+Wire Wire Line
+	4600 7150 4700 7150
+Wire Wire Line
+	4700 7350 4700 7450
+$Comp
+L Connector:Conn_01x05_Female J2
 U 1 1 5D1D79FB
 P 4400 7250
 F 0 "J2" H 4294 6925 50  0000 C CNN
-F 1 "Conn_01x03_Female" H 4294 7016 50  0000 C CNN
-F 2 "Connector_PinSocket_2.54mm:PinSocket_1x03_P2.54mm_Vertical_SMD_Pin1Left" H 4400 7250 50  0001 C CNN
+F 1 "Conn_01x05_Female" H 4294 7016 50  0000 C CNN
+F 2 "Connector_PinSocket_2.54mm:PinSocket_1x05_P2.54mm_Vertical_SMD_Pin1Left" H 4400 7250 50  0001 C CNN
 F 3 "~" H 4400 7250 50  0001 C CNN
 	1    4400 7250
@@
 $EndComp
 Wire Wire Line
-	4700 7250 4700 7150
-Wire Wire Line
-	4600 7150 4700 7150
-Wire Wire Line
-	4700 7350 4700 7550
+	4600 7450 4700 7450
+Connection ~ 4700 7450
+Wire Wire Line
+	4700 7450 4700 7550
+Wire Wire Line
+	4600 7050 4700 7050
+Wire Wire Line
+	4700 7050 4700 7150
+Connection ~ 4700 7150
 $EndSCHEMATC

Commit message: :recycle: rerouted all pcb
same


same
Connections:
- net GND: no longer J9.2 (Pin_2), J9.4 (Pin_4)
- no-connect marks 28 -> 30
Changed lines of the file:
@@
-$EndComp
-$Comp
-L power:GND #PWR0137
-U 1 1 5D1B3580
-P 3000 7450
-F 0 "#PWR0137" H 3000 7200 50  0001 C CNN
-F 1 "GND" V 3005 7322 50  0000 R CNN
-F 2 "" H 3000 7450 50  0001 C CNN
-F 3 "" H 3000 7450 50  0001 C CNN
-	1    3000 7450
-	0    1    1    0
-$EndComp
-$Comp
-L power:GND #PWR0138
-U 1 1 5D1B35E5
-P 3000 7250
-F 0 "#PWR0138" H 3000 7000 50  0001 C CNN
-F 1 "GND" V 3005 7122 50  0000 R CNN
-F 2 "" H 3000 7250 50  0001 C CNN
-F 3 "" H 3000 7250 50  0001 C CNN
-	1    3000 7250
-	0    1    1    0
 $EndComp
 $Comp
@@
 	3000 7150 3100 7150
 Wire Wire Line
-	3100 7250 3000 7250
-Wire Wire Line
 	3000 7350 3100 7350
-Wire Wire Line
-	3100 7450 3000 7450
 Wire Wire Line
 	3000 7550 3100 7550
@@
 	4700 7050 4700 7150
 Connection ~ 4700 7150
+NoConn ~ 3100 7250
+NoConn ~ 3100 7450
 $EndSCHEMATC

Commit message: :zap: Added Either way power and more rugged fixations
same
Parts:
- removed D1, D2: 1N5819, Diode_SMD:D_SOD-123, symbol Diode:1N5819
- added D1: MB1S, NN_Footprints:SOIC-4-POWER, symbol Device:D_Bridge_+-AA
- added H1, H2: MountingHole, MountingHole:MountingHole_2.7mm_M2.5, symbol Mechanical:MountingHole
Connections:
- net +12V: now also D1.1 (+)
- net -12V: now also D1.2 (-)
- net at J1.1 (Pin_1), J1.2 (Pin_2): now also D1.4 (~~)
- net at J1.10 (Pin_10), J1.9 (Pin_9): now also D1.3 (~~)
Other:
- moved on the sheet: J1, J2, J9

Commit message: :recycle: Redid routing
same


same


same
Connections:
- net GND: no longer J2.4 (Pin_4), J2.5 (Pin_5), R1.1, U3.3 (+), U3.5 (+)
- new net GNDA: J2.4 (Pin_4), J2.5 (Pin_5), R1.1, U3.3 (+), U3.5 (+)
Changed lines of the file:
@@
 Text GLabel 9550 5100 1    50   Input ~ 0
 AUDIO_OUT
-$Comp
-L power:GND #PWR0109
-U 1 1 5D197FFF
-P 8750 5000
-F 0 "#PWR0109" H 8750 4750 50  0001 C CNN
-F 1 "GND" V 8755 4872 50  0000 R CNN
-F 2 "" H 8750 5000 50  0001 C CNN
-F 3 "" H 8750 5000 50  0001 C CNN
-	1    8750 5000
-	0    1    1    0
-$EndComp
 Wire Wire Line
 	8800 5000 8750 5000
-$Comp
-L power:GND #PWR0110
-U 1 1 5D199726
-P 7550 5100
-F 0 "#PWR0110" H 7550 4850 50  0001 C CNN
-F 1 "GND" V 7555 4972 50  0000 R CNN
-F 2 "" H 7550 5100 50  0001 C CNN
-F 3 "" H 7550 5100 50  0001 C CNN
-	1    7550 5100
-	0    1    1    0
-$EndComp
 Wire Wire Line
 	7550 5100 7600 5100
@@
 	1    6900 5450
 	-1   0    0    1
-$EndComp
-$Comp
-L power:GND #PWR0111
-U 1 1 5D1A3A01
-P 6900 5700
-F 0 "#PWR0111" H 6900 5450 50  0001 C CNN
-F 1 "GND" H 6905 5527 50  0000 C CNN
-F 2 "" H 6900 5700 50  0001 C CNN
-F 3 "" H 6900 5700 50  0001 C CNN
-	1    6900 5700
-	1    0    0    -1
 $EndComp
 Wire Wire Line
@@
 Wire Wire Line
 	3500 7250 3500 7350
-Connection ~ 3500 7250
 Wire Wire Line
 	3500 7250 3400 7250
@@
 Connection ~ 3500 7350
 Wire Wire Line
-	3500 7250 3500 7150
-Wire Wire Line
-	3400 7150 3500 7150
-Wire Wire Line
 	3500 7350 3500 7450
+Wire Wire Line
+	3400 7450 3500 7450
+Connection ~ 3500 7450
+Wire Wire Line
+	3500 7450 3500 7550
+NoConn ~ 1900 7250
+NoConn ~ 1900 7450
+$Comp
+L Mechanical:MountingHole H1
+U 1 1 5EFA71F2
+P 9950 2050
+F 0 "H1" H 10050 2096 50  0000 L CNN
+F 1 "MountingHole" H 10050 2005 50  0000 L CNN
+F 2 "MountingHole:MountingHole_2.7mm_M2.5" H 9950 2050 50  0001 C CNN
+F 3 "~" H 9950 2050 50  0001 C CNN
+	1    9950 2050
+	1    0    0    -1
+$EndComp
+$Comp
+L Mechanical:MountingHole H2
+U 1 1 5EFA78E3
+P 9950 2375
+F 0 "H2" H 10050 2421 50  0000 L CNN
+F 1 "MountingHole" H 10050 2330 50  0000 L CNN
+F 2 "MountingHole:MountingHole_2.7mm_M2.5" H 9950 2375 50  0001 C CNN
+F 3 "~" H 9950 2375 50  0001 C CNN
+	1    9950 2375
+	1    0    0    -1
+$EndComp
+$Comp
+L Device:D_Bridge_+-AA D1
+U 1 1 5F016EBA
+P 5950 7000
+F 0 "D1" V 5996 6656 50  0000 R CNN
+F 1 "MB1S" V 5905 6656 50  0000 R CNN
+F 2 "NN_Footprints:SOIC-4-POWER" H 5950 7000 50  0001 C CNN
+F 3 "~" H 5950 7000 50  0001 C CNN
+	1    5950 7000
+	0    -1   -1   0
+$EndComp
+Wire Wire Line
+	5950 6575 5950 6700
+Wire Wire Line
+	5950 7300 5950 7400
+Wire Wire Line
+	5650 7000 5650 6800
+Wire Wire Line
+	5150 6800 5650 6800
+Wire Wire Line
+	5250 7200 5150 7200
+Wire Wire Line
+	6250 7000 6250 7600
+Wire Wire Line
+	6250 7600 5250 7600
+Wire Wire Line
+	5250 7600 5250 7200
+$Comp
+L power:GNDA #PWR0109
+U 1 1 5EFB42E6
+P 8750 5000
+F 0 "#PWR0109" H 8750 4750 50  0001 C CNN
+F 1 "GNDA" V 8755 4873 50  0000 R CNN
+F 2 "" H 8750 5000 50  0001 C CNN
+F 3 "" H 8750 5000 50  0001 C CNN
+	1    8750 5000
+	0    1    1    0
+$EndComp
+$Comp
+L power:GNDA #PWR0110
+U 1 1 5EFB94C2
+P 7550 5100
+F 0 "#PWR0110" H 7550 4850 50  0001 C CNN
+F 1 "GNDA" V 7555 4973 50  0000 R CNN
+F 2 "" H 7550 5100 50  0001 C CNN
+F 3 "" H 7550 5100 50  0001 C CNN
+	1    7550 5100
+	0    1    1    0
+$EndComp
+$Comp
+L power:GNDA #PWR0111
+U 1 1 5EFBA343
+P 6900 5700
+F 0 "#PWR0111" H 6900 5450 50  0001 C CNN
+F 1 "GNDA" H 6905 5527 50  0000 C CNN
+F 2 "" H 6900 5700 50  0001 C CNN
+F 3 "" H 6900 5700 50  0001 C CNN
+	1    6900 5700
+	1    0    0    -1
+$EndComp
+$Comp
+L power:GNDA #PWR?
+U 1 1 5EFCAB21
+P 3500 7050
+F 0 "#PWR?" H 3500 6800 50  0001 C CNN
+F 1 "GNDA" V 3505 6922 50  0000 R CNN
+F 2 "" H 3500 7050 50  0001 C CNN
+F 3 "" H 3500 7050 50  0001 C CNN
+	1    3500 7050
+	0    -1   -1   0
+$EndComp
 $Comp
 L Connector:Conn_01x05_Female J2
@@
 $EndComp
 Wire Wire Line
-	3400 7450 3500 7450
-Connection ~ 3500 7450
-Wire Wire Line
-	3500 7450 3500 7550
-Wire Wire Line
-	3400 7050 3500 7050
-Wire Wire Line
-	3500 7050 3500 7150
-Connection ~ 3500 7150
-NoConn ~ 1900 7250
-NoConn ~ 1900 7450
-$Comp
-L Mechanical:MountingHole H1
-U 1 1 5EFA71F2
-P 9950 2050
-F 0 "H1" H 10050 2096 50  0000 L CNN
-F 1 "MountingHole" H 10050 2005 50  0000 L CNN
-F 2 "MountingHole:MountingHole_2.7mm_M2.5" H 9950 2050 50  0001 C CNN
-F 3 "~" H 9950 2050 50  0001 C CNN
-	1    9950 2050
-	1    0    0    -1
-$EndComp
-$Comp
-L Mechanical:MountingHole H2
-U 1 1 5EFA78E3
-P 9950 2375
-F 0 "H2" H 10050 2421 50  0000 L CNN
-F 1 "MountingHole" H 10050 2330 50  0000 L CNN
-F 2 "MountingHole:MountingHole_2.7mm_M2.5" H 9950 2375 50  0001 C CNN
-F 3 "~" H 9950 2375 50  0001 C CNN
-	1    9950 2375
-	1    0    0    -1
-$EndComp
-$Comp
-L Device:D_Bridge_+-AA D1
-U 1 1 5F016EBA
-P 5950 7000
-F 0 "D1" V 5996 6656 50  0000 R CNN
-F 1 "MB1S" V 5905 6656 50  0000 R CNN
-F 2 "NN_Footprints:SOIC-4-POWER" H 5950 7000 50  0001 C CNN
-F 3 "~" H 5950 7000 50  0001 C CNN
-	1    5950 7000
-	0    -1   -1   0
-$EndComp
-Wire Wire Line
-	5950 6575 5950 6700
-Wire Wire Line
-	5950 7300 5950 7400
-Wire Wire Line
-	5650 7000 5650 6800
-Wire Wire Line
-	5150 6800 5650 6800
-Wire Wire Line
-	5250 7200 5150 7200
-Wire Wire Line
-	6250 7000 6250 7600
-Wire Wire Line
-	6250 7600 5250 7600
-Wire Wire Line
-	5250 7600 5250 7200
+	3500 7050 3400 7050
+Wire Wire Line
+	3400 7150 3500 7150
+Wire Wire Line
+	3500 7150 3500 7050
+Connection ~ 3500 7050
 $EndSCHEMATC
