File: quadrants/Front.sch (KiCad schematic (older format))
At the start: 32 parts, among them CON1 microSD_Card, J12 Conn_01x05_Male, J17 Conn_01x05_Male, J5 TIME_CV, J6 CHANNEL_CV, J7 RESET_CV, J8 OUT, SW1 SW_Push_LED, X1 50k, Y1 50k

Commit message: :construction: prepare 4 layer board layout
Parts:
- removed C10, C11, C12, C9: 10nF, Capacitor_SMD:C_0603_1608Metric, symbol Device:C_Small
- removed J12, J17: Conn_01x05_Male, Connector_PinHeader_2.54mm:PinHeader_1x05_P2.54mm_Vertical, symbol Connector:Conn_01x05_Male
- X1, Y1: symbol Device:R_POT -> quadrants-rescue:R_POT-Device
Connections:
- net GNDA is gone; now on net GND: J8.S
- no-connect marks 4 -> 2
Other:
- moved on the sheet: R13, R14, R15, R16

Commit message: :construction: first draft at 4 layer layout
same
Parts:
- X1, Y1: symbol quadrants-rescue:R_POT-Device -> quadrants-rescue:R_POT-Device-quadrants-rescue
Changed lines of the file:
@@
 RESET_SW
 $Comp
-L quadrants-rescue:R_POT-Device X1
+L quadrants-rescue:R_POT-Device-quadrants-rescue X1
 U 1 1 5D281D3E
 P 1350 2750
@@
 	1550 2750 1500 2750
 $Comp
-L quadrants-rescue:R_POT-Device Y1
+L quadrants-rescue:R_POT-Device-quadrants-rescue Y1
 U 1 1 5D282FDC
 P 1400 4250
