File: quadrants/quadrants.kicad_pcb (KiCad board)
At the start: 2 copper layers, 107.5 x 41.3 mm, 57 parts, among them CON1 microSD_Card, J1 POWER, J12 Conn_01x05_Male, J17 Conn_01x05_Male, J2 Conn_01x05_Female, J5 TIME_CV, J6 CHANNEL_CV, J7 RESET_CV, J8 OUT, J9 Conn_01x05_Female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

Commit message: :lipstick: Add BLM logo
same
Parts:
- added G***: LOGO, NN_Footprints:blm_small, B.Cu at (152.4, 64.9)
Other:
- board text added: "quadrants main board v1.0 - CC-BY-SA-3.0"
- board text removed: "quadrants main board v1.0"

Commit message: :construction: prepare 4 layer board layout
Parts:
- removed C10, C11, C12, C9: 10nF, Capacitor_SMD:C_0603_1608Metric
- removed G***: LOGO, NN_Footprints:blm_small
- removed G*** (x2): LOGO, NN_Footprints:nebularnoise_logo
- removed G***: LOGO, NN_Footprints:caution_hot
- removed J12, J17: Conn_01x05_Male, Connector_PinHeader_2.54mm:PinHeader_1x05_P2.54mm_Vertical
- removed J2, J9: Conn_01x05_Female, Connector_PinSocket_2.54mm:PinSocket_1x05_P2.54mm_Vertical_SMD_Pin1Left
- added H1: MountingHole, MountingHole:MountingHole_2.7mm_M2.5, F.Cu at (83.6, 27.3)
- added H2: MountingHole, MountingHole:MountingHole_2.7mm_M2.5, F.Cu at (90.5, 27.3)
- moved D2 81.7 mm to (107.0, 64.2), turned to 270 degrees
- moved R11 76.0 mm to (104.2, 64.5), turned to 270 degrees
- moved R10 74.6 mm to (102.5, 64.5), turned to 90 degrees
- moved R6 72.5 mm to (119.0, 62.7), turned to 90 degrees
- moved R8 71.0 mm to (120.6, 62.8), turned to 270 degrees
- moved R18 69.4 mm to (105.5, 68.2)
- moved U2 66.1 mm to (129.0, 64.8), turned to 0 degrees
- moved R7 62.5 mm to (136.8, 89.5)
- moved R9 62.5 mm to (135.3, 91.3)
- moved C1 58.0 mm to (138.0, 84.2)
- moved C5 42.8 mm to (173.2, 69.0), turned to 90 degrees
- moved C4 35.5 mm to (166.0, 61.8), turned to 90 degrees
- moved J1 12.0 mm to (121.5, 48.5), turned to 180 degrees
- moved C7 11.0 mm to (177.0, 62.2)
- moved R5 9.49 mm to (168.5, 62.5), turned to 0 degrees
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Connections:
- J8 pad S: GNDA -> GND
- R1 pad 1: GNDA -> GND
- U3 pad 3: GNDA -> GND
- U3 pad 5: GNDA -> GND
Routing:
- net +3V3: track 99.2 -> 0.00 mm, vias 2 -> 0
- net +5V: track 95.9 -> 0.00 mm, vias 3 -> 0
- net Net-(J5-PadT): track 88.9 -> 0.00 mm, vias 4 -> 0
- net Net-(J7-PadT): track 85.3 -> 0.00 mm, vias 4 -> 0
- net GNDA: track 85.2 -> 0.00 mm, vias 6 -> 0
- net Net-(J8-PadT): track 84.2 -> 0.00 mm
- net GND: track 92.7 -> 8.51 mm, vias 10 -> 8
- net -12V: track 82.7 -> 0.00 mm, vias 2 -> 0
- net Net-(J6-PadT): track 82.6 -> 0.00 mm, vias 4 -> 0
- net +12V: track 73.9 -> 0.00 mm, vias 6 -> 0
- net RESET_SW: track 51.3 -> 0.00 mm
- net SS: track 50.7 -> 0.00 mm
- net MOSI: track 50.6 -> 0.00 mm
- net MISO: track 50.0 -> 0.00 mm
- net SCLK: track 50.0 -> 0.00 mm
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- added copper zone on In2.Cu, net GND
- removed copper zone on B.Cu, net +12V
- removed copper zone on F.Cu, net +12V
- removed copper zone on B.Cu, net GND
- removed copper zone on F.Cu, net GND
- removed copper zone on B.Cu, net GNDA
- removed copper zone on F.Cu, net GNDA
- removed copper zone on B.Cu, net Net-(HS1-Pad1)
- removed copper zone on F.Cu, net Net-(HS1-Pad1)
Other:
- board size 107.5 x 41.3 mm -> 107.5 x 41 mm
- copper layers 2 -> 4

Commit message: :construction: first draft at 4 layer layout
same
Parts:
- removed C6: 10uF, Capacitor_SMD:CP_Elec_5x5.9
- removed H1, H2: MountingHole, MountingHole:MountingHole_2.7mm_M2.5
- C2, C3, D1, U4: moved to B.Cu
- J1: footprint Connector_PinHeader_2.54mm:PinHeader_2x05_P2.54mm_Horizontal -> Connector_PinHeader_2.54mm:PinHeader_2x05_P2.54mm_Vertical_SMD; moved to B.Cu
- moved U4 52.0 mm to (193.2, 65.0), turned to 180 degrees
- moved R7 35.7 mm to (109.7, 66.2)
- moved R9 34.8 mm to (109.7, 67.8)
- moved C3 34.0 mm to (160.2, 64.8), turned to 270 degrees
- moved C1 31.2 mm to (112.0, 67.0), turned to 270 degrees
- moved D1 29.7 mm to (120.5, 65.2), turned to 90 degrees
- moved C2 28.8 mm to (151.8, 66.0), turned to 90 degrees
- moved J1 20.2 mm to (133.5, 64.8)
- moved U2 13.8 mm to (115.2, 64.7), turned to 270 degrees
- moved R8 9.32 mm to (111.2, 62.5), turned to 0 degrees
- moved R6 7.90 mm to (111.2, 64.0), turned to 180 degrees
- moved D2 3.92 mm to (103.8, 66.5), turned to 180 degrees
- moved R10 2.78 mm to (103.8, 62.0), turned to 0 degrees
- moved C7 2.75 mm to (177.0, 65.0)
- moved R18 1.98 mm to (104.5, 70.0)
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Routing:
- net +3V3: track 0.00 -> 128.4 mm, vias 0 -> 2
- net CHANNEL_CV_ADC: track 0.00 -> 99.3 mm, vias 0 -> 2
- net +12V: track 0.00 -> 87.9 mm, vias 0 -> 8
- net RESET_CV: track 0.00 -> 87.1 mm, vias 0 -> 2
- net TIME_CV_ADC: track 0.00 -> 83.1 mm
- net -12V: track 0.00 -> 75.1 mm, vias 0 -> 4
- net AUDIO_OUT: track 0.00 -> 74.0 mm
- net MOSI: track 0.00 -> 54.4 mm
- net SS: track 0.00 -> 48.5 mm, vias 0 -> 1
- net RESET_SW: track 0.00 -> 44.0 mm, vias 0 -> 1
- net TIME_POT: track 0.00 -> 38.0 mm
- net LED_RESET: track 0.00 -> 37.0 mm, vias 0 -> 1
- net MISO: track 0.00 -> 36.5 mm
- net A4: track 0.00 -> 33.7 mm
- net A2: track 0.00 -> 33.1 mm
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- added copper zone on B.Cu, net +12V
- added copper zone on In1.Cu, net +12V
- added copper zone on B.Cu, net GND
- added copper zone on B.Cu, net Net-(HS1-Pad1)
Other:
- board size 107.5 x 41 mm -> 107.5 x 19.5 mm
- board text added: "quadrants main board v2.0BETA - CC-BY-SA-3.0"
- board text removed: "CAUTION HOT"
- board text removed: "Quadrants"
- board text removed: "github.com /nebularnoise /quadrants"
- board text removed: "quadrants main board v1.0 - CC-BY-SA-3.0"
- board text removed: "quadrants power board v1.0"
