File: quadrants/quadrants.kicad_pcb (KiCad board)
At the start: 4 copper layers, 107.5 x 19.5 mm, 45 parts, among them CON1 microSD_Card, J1 POWER, J5 TIME_CV, J6 CHANNEL_CV, J7 RESET_CV, J8 OUT, SW1 SW_Push_LED, U1 Teensy3.2, U2 MCP6002, U3 TL072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

Commit message: :recycle: Use THT power header !
Parts:
- J1: footprint Connector_PinHeader_2.54mm:PinHeader_2x05_P2.54mm_Vertical_SMD -> Connector_PinHeader_2.54mm:PinHeader_2x05_P2.54mm_Vertical
- moved J1 4.83 mm to (133.5, 59.9)
Routing:
- net MISO: track 36.5 -> 41.0 mm
- net LED_RESET: track 37.0 -> 41.1 mm
- net +3V3: track 128.4 -> 132.4 mm
- net Net-(D1-Pad4): track 20.3 -> 17.2 mm
- net SS: track 48.5 -> 51.2 mm
- net MOSI: track 54.4 -> 57.0 mm
- net Net-(D1-Pad3): track 21.2 -> 19.6 mm
- net GND: track 35.7 -> 36.1 mm, vias 45 -> 32
Other:
- board text added: "POWER"
